Commit message: fixed file paths

File: my-models/niryo_one_description/urdf/v2/niryo_one.urdf (robot description, URDF)
Before this commit: robot niryo_one, 9 links, 8 joints
Links:
- link arm_link: geometry collision mesh filename=../../../niryo_one_description/meshes/v2/stl/arm_link.stl; visual mesh filename=../../../niryo_one_description/meshes/v2/collada/arm_link.d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
- link base_link: geometry collision mesh filename=../../../niryo_one_description/meshes/v2/stl/base_link.stl; visual mesh filename=../../../niryo_one_description/meshes/v2/collada/base_link.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
- link elbow_link: geometry collision mesh filename=../../../niryo_one_description/meshes/v2/stl/elbow_link.stl; visual mesh filename=../../../niryo_one_description/meshes/v2/collada/elbow_link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
- link forearm_link: geometry collision mesh filename=../../../niryo_one_description/meshes/v2/stl/forearm_link.s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; visual mesh filename=../../../niryo_one_description/meshes/v2/collada/forearm_li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
- link hand_link: geometry collision mesh filename=../../../niryo_one_description/meshes/v2/stl/hand_link.stl; visual mesh filename=../../../niryo_one_description/meshes/v2/collada/hand_link.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
- link shoulder_link: geometry collision mesh filename=../../../niryo_one_description/meshes/v2/stl/shoulder_link.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; visual mesh filename=../../../niryo_one_description/meshes/v2/collada/shoulder_l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
- link wrist_link: geometry collision mesh filename=../../../niryo_one_description/meshes/v2/stl/wrist_link.stl; visual mesh filename=../../../niryo_one_description/meshes/v2/collada/wrist_link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
